File: projects/Switch transistor IRL540N/schema.brd (EAGLE design)
At the start: 160 x 100 mm, 6 parts, among them Q1 IRF3704L-V

Commit message: rinominato progetto switch.
Parts:
- Q1: value IRF3704L-V -> IRL540N
- R1, R2: device resistor-power:AC01 -> resistor-power:RS1/4
- moved CMD 26.2 mm to (25.4, 7.62), turned to 180 degrees
- moved Q1 23.2 mm to (6.35, 17.8), turned to 0 degrees
- moved R2 14.2 mm to (26.7, 15.2), turned to 90 degrees
- moved R1 8.52 mm to (24.1, 15.2), turned to 90 degrees
- moved LED 5.39 mm to (6.35, 7.62)
- moved 12VDC 5.39 mm to (16.5, 7.62)
Routing:
- net N$2: track 11.5 -> 25.4 mm, vias 0 -> 8
- net N$6: track 6.40 -> 20.3 mm, vias 0 -> 3
- net N$3: track 9.14 -> 2.54 mm
- net N$5: track 19.2 -> 12.6 mm, vias 0 -> 4
- net N$1: track 6.34 -> 2.54 mm
Other:
- board size 160 x 100 mm -> 27.9 x 21.3 mm

Commit message: in lavoro alimentatore
Connections:
- removed net N$3: CMD.1, R2.1
- removed net N$6: 12VDC.2, Q1.3
- new net GND: 12VDC.2, CMD.1, Q1.3, R2.1
Routing:
- net GND: track 0.00 -> 22.8 mm, vias 0 -> 3
- net N$6: track 20.3 -> 0.00 mm, vias 3 -> 0
- net N$27: track 0.00 -> 15.2 mm, vias 1 -> 0
- net N$3: track 2.54 -> 0.00 mm
Changed lines of the file:
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@@
 <drawing>
 <settings>
-<setting alwaysvectorfont="yes"/>
+<setting alwaysvectorfont="no"/>
 <setting verticaltext="up"/>
 </settings>
@@
 <via x="21.59" y="20.32" extent="1-16" drill="0.35"/>
 </signal>
-<signal name="N$3">
-<contactref element="CMD" pad="1"/>
-<contactref element="R2" pad="1"/>
-<wire x1="26.67" y1="10.16" x2="26.67" y2="7.62" width="0.1524" layer="16"/>
-</signal>
 <signal name="N$4">
 <contactref element="12VDC" pad="1"/>
@@
 <wire x1="13.9954" y1="3.81" x2="13.9954" y2="7.62" width="0.1524" layer="16"/>
 <wire x1="3.8354" y1="3.81" x2="13.9954" y2="3.81" width="0.1524" layer="16"/>
-</signal>
-<signal name="N$6">
-<contactref element="12VDC" pad="2"/>
-<contactref element="Q1" pad="3"/>
-<wire x1="8.89" y1="17.78" x2="11.43" y2="17.78" width="0.1524" layer="16"/>
-<wire x1="11.43" y1="17.78" x2="13.97" y2="17.78" width="0.1524" layer="16"/>
-<wire x1="13.97" y1="17.78" x2="16.51" y2="17.78" width="0.1524" layer="16"/>
-<wire x1="16.51" y1="17.78" x2="18.9992" y2="17.78" width="0.1524" layer="16"/>
-<wire x1="18.9992" y1="17.78" x2="18.9992" y2="7.62" width="0.1524" layer="16"/>
-<via x="11.43" y="17.78" extent="1-16" drill="0.35"/>
-<via x="13.97" y="17.78" extent="1-16" drill="0.35"/>
-<via x="16.51" y="17.78" extent="1-16" drill="0.35"/>
 </signal>
 <signal name="N$5">
@@
 <via x="16.51" y="10.16" extent="1-16" drill="0.35"/>
 </signal>
-<signal name="N$14">
-<via x="19.05" y="10.16" extent="1-16" drill="0.35"/>
-</signal>
 <signal name="N$15">
 <via x="21.59" y="10.16" extent="1-16" drill="0.35"/>
@@
 <via x="16.51" y="12.7" extent="1-16" drill="0.35"/>
 </signal>
-<signal name="N$23">
-<via x="19.05" y="12.7" extent="1-16" drill="0.35"/>
-</signal>
 <signal name="N$24">
 <via x="21.59" y="12.7" extent="1-16" drill="0.35"/>
@@
 </signal>
 <signal name="N$27">
-<via x="19.05" y="17.78" extent="1-16" drill="0.35"/>
-</signal>
-<signal name="N$28">
-<via x="19.05" y="15.24" extent="1-16" drill="0.35"/>
+<wire x1="19.05" y1="17.78" x2="26.67" y2="17.78" width="0.1524" layer="16"/>
+<wire x1="26.67" y1="17.78" x2="26.67" y2="10.16" width="0.1524" layer="16"/>
 </signal>
 <signal name="N$29">
@@
 <via x="16.51" y="7.62" extent="1-16" drill="0.35"/>
 </signal>
-<signal name="N$48">
-<via x="26.67" y="12.7" extent="1-16" drill="0.35"/>
-</signal>
-<signal name="N$49">
-<via x="26.67" y="15.24" extent="1-16" drill="0.35"/>
-</signal>
 <signal name="N$50">
 <via x="24.13" y="15.24" extent="1-16" drill="0.35"/>
@@
 <via x="24.13" y="12.7" extent="1-16" drill="0.35"/>
 </signal>
-<signal name="N$39">
-<via x="26.67" y="17.78" extent="1-16" drill="0.35"/>
-</signal>
 <signal name="N$47">
 <via x="24.13" y="17.78" extent="1-16" drill="0.35"/>
 </signal>
+<signal name="GND">
+<contactref element="CMD" pad="1"/>
+<contactref element="R2" pad="1"/>
+<wire x1="26.67" y1="10.16" x2="26.67" y2="7.62" width="0.1524" layer="16"/>
+<contactref element="12VDC" pad="2"/>
+<contactref element="Q1" pad="3"/>
+<wire x1="8.89" y1="17.78" x2="11.43" y2="17.78" width="0.1524" layer="16"/>
+<wire x1="11.43" y1="17.78" x2="13.97" y2="17.78" width="0.1524" layer="16"/>
+<wire x1="13.97" y1="17.78" x2="16.51" y2="17.78" width="0.1524" layer="16"/>
+<wire x1="16.51" y1="17.78" x2="18.9992" y2="17.78" width="0.1524" layer="16"/>
+<wire x1="18.9992" y1="17.78" x2="18.9992" y2="7.62" width="0.1524" layer="16"/>
+<via x="11.43" y="17.78" extent="1-16" drill="0.35"/>
+<via x="13.97" y="17.78" extent="1-16" drill="0.35"/>
+<via x="16.51" y="17.78" extent="1-16" drill="0.35"/>
+<wire x1="18.9992" y1="7.62" x2="26.67" y2="7.62" width="0" layer="19" extent="1-1"/>
+</signal>
 </signals>
