File: projects/Alimentatore_Banco/Regolatori_LM317.brd (EAGLE design)
At the start: 160 x 100 mm, 20 parts

Commit message: terminato schema regolatori.
Parts:
- removed LM317-1, LM317-2, LM317-3: (no value), v-reg:TO220V
- added LM317-12, LM317-24, LM317-5: (no value), v-reg:TO220V
- C1, C2, C3, C4: device rcl:E2-5 -> rcl:C025-025X050
- R1, R4, R6: device resistor:RTRIM3339P -> rcl:RTRIM64W
- moved R6 112.1 mm to (58.4, 61.0), turned to 270 degrees
- moved D3 100.1 mm to (59.7, 67.3), turned to 180 degrees
- moved C2 98.0 mm to (44.5, 72.4)
- moved R4 92.1 mm to (45.7, 61.0), turned to 270 degrees
- moved 24V 91.5 mm to (38.1, 52.1)
- moved 12V 90.4 mm to (48.3, 52.1)
- moved 5V 89.3 mm to (58.4, 52.1)
- moved R5 87.9 mm to (59.7, 64.8), turned to 180 degrees
- moved C4 87.2 mm to (57.1, 72.4)
- moved R2 80.0 mm to (34.3, 64.8), turned to 180 degrees
- moved D2 78.0 mm to (47.0, 67.3), turned to 180 degrees
- moved R1 73.0 mm to (33.0, 61.0), turned to 270 degrees
- moved R3 65.1 mm to (47.0, 64.8), turned to 180 degrees
- moved C1 62.7 mm to (25.4, 61.0), turned to 270 degrees
- moved D1 56.4 mm to (34.3, 67.3), turned to 180 degrees
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Connections:
- net GND: now also C1.2, C2.2, C3.2, C4.2; no longer C1.-, C2.-, C3.-, C4.-
- net N$1: now also LM317-24.2; no longer LM317-2.2
- net N$4: now also C2.1, LM317-12.1; no longer C2.+, LM317-1.1
- net N$5: now also LM317-12.2; no longer LM317-1.2
- net N$6: now also C4.1, LM317-5.1; no longer C4.+, LM317-3.1
- net N$7: now also LM317-5.2; no longer LM317-3.2
- net N$9: now also C3.1, LM317-24.1; no longer C3.+, LM317-2.1
- net VCC: now also C1.1, LM317-12.3, LM317-24.3, LM317-5.3; no longer C1.+, LM317-1.3, LM317-2.3, LM317-3.3
Routing:
- net GND: track 0.00 -> 125.1 mm
- net VCC: track 0.00 -> 76.2 mm
- net N$7: track 0.00 -> 33.1 mm
- net N$1: track 0.00 -> 33.0 mm
- net N$5: track 0.00 -> 30.5 mm
- net N$9: track 0.00 -> 17.8 mm
- net N$6: track 0.00 -> 17.8 mm
- net N$4: track 0.00 -> 17.8 mm
Other:
- board size 160 x 100 mm -> 48.3 x 40.6 mm
