File: projects/Alimentatore_Banco/Regolatori_LM317.sch (EAGLE design)
At the start: 20 parts

Commit message: terminato schema regolatori.
Parts:
- C1, C2, C3, C4: device rcl:CPOL-EUE2-5 -> rcl:C-EU025-025X050
- R1, R4, R6: device resistor:R-TRIMM3339P -> rcl:R-TRIMM64W
- renumbered LM317-1 to LM317-12, LM317-2 to LM317-24, LM317-3 to LM317-5
Connections:
- net GND: now also C1.2, C2.2, C3.2, C4.2; no longer C1.-, C2.-, C3.-, C4.-
- net N$4: now also C2.1; no longer C2.+
- net N$6: now also C4.1; no longer C4.+
- net N$9: now also C3.1; no longer C3.+
- net VCC: now also C1.1; no longer C1.+
